File: V5.9aSMD.brd (EAGLE design)
At the start: 85.1 x 50.8 mm, 38 parts

Commit message: Production files
Routing:
- net N$16: track 15.2 -> 10.2 mm
Other:
- board text added: "V5.9"
Changed lines of the file:
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@@
 <text x="64.516" y="4.572" size="1.4224" layer="21" rot="R90">Load/Test</text>
 <text x="83.312" y="6.858" size="1.4224" layer="21" rot="R90">Boost</text>
+<text x="12.7" y="1.27" size="1.778" layer="26" rot="MR0">V5.9</text>
 </plain>
 <attributes>
@@
 <wire x1="47.94" y1="17.78" x2="49.53" y2="17.78" width="0.4064" layer="1"/>
 <wire x1="49.53" y1="17.78" x2="49.53" y2="21.463" width="0.4064" layer="1"/>
-<wire x1="47.94" y1="13.5032" x2="47.94" y2="17.78" width="0.4064" layer="1"/>
+<wire x1="47.94" y1="12.9952" x2="47.94" y2="17.78" width="0.4064" layer="1"/>
 <wire x1="49.53" y1="17.78" x2="59.69" y2="17.78" width="0.4064" layer="1"/>
 <wire x1="59.69" y1="20.64" x2="59.69" y2="17.78" width="0.4064" layer="1"/>
 <contactref element="S4" pad="3"/>
-<wire x1="47.94" y1="13.5032" x2="43.0276" y2="13.5032" width="0.4064" layer="1"/>
-<wire x1="43.0276" y1="13.5032" x2="43.0276" y2="12.9032" width="0.4064" layer="1"/>
+<wire x1="47.94" y1="12.9952" x2="43.0276" y2="12.9952" width="0.4064" layer="1"/>
+<wire x1="43.0276" y1="12.9952" x2="43.0276" y2="12.9032" width="0.4064" layer="1"/>
 <contactref element="U$1" pad="10"/>
 <wire x1="49.53" y1="21.463" x2="51.082" y2="21.463" width="0.4064" layer="1"/>
@@
 <contactref element="C11" pad="2"/>
 <contactref element="S1" pad="3"/>
-<wire x1="52.07" y1="4.13" x2="60.96" y2="4.13" width="0.4064" layer="1"/>
-<wire x1="60.96" y1="4.13" x2="58.42" y2="4.1768" width="0.4064" layer="1"/>
+<wire x1="52.07" y1="4.13" x2="58.42" y2="4.13" width="0.4064" layer="1"/>
+<wire x1="58.42" y1="4.13" x2="58.42" y2="4.1768" width="0.4064" layer="1"/>
 <wire x1="52.07" y1="4.13" x2="48.26" y2="4.13" width="0.4064" layer="1"/>
 </signal>
@@
 <contactref element="C10" pad="-"/>
 <contactref element="C12" pad="1"/>
-<polygon width="0.4064" layer="16" spacing="0.3048" isolate="0.3048">
+<polygon width="0.4064" layer="16" spacing="0.3048" isolate="0.6096">
 <vertex x="0" y="-1.27"/>
 <vertex x="0" y="53.34"/>
@@
 <vertex x="86.36" y="-1.27"/>
 </polygon>
-<polygon width="0.4064" layer="1" spacing="0.3048" isolate="0.3048">
-<vertex x="-2.54" y="-2.54"/>
-<vertex x="-2.54" y="53.34"/>
+<polygon width="0.4064" layer="1" spacing="0.3048" isolate="0.6096">
+<vertex x="-3.81" y="-2.54"/>
+<vertex x="-3.81" y="53.34"/>
 <vertex x="88.9" y="53.34"/>
 <vertex x="88.9" y="-2.54"/>
